Commit message: env update

File: turtlebot_env/resources/obstacle.urdf (robot description, URDF)
Before this commit: robot obstacle, 1 links, 0 joints
Links:
- link base_link: geometry collision cylinder length=0.3 radius=0.17; visual cylinder length=0.3 radius=0.17

Commit message: update

File: turtlebot_env/resources/obstacle.urdf (robot description, URDF)
Before this commit: robot obstacle, 1 links, 0 joints
Links:
- link base_link: geometry collision cylinder length=0 radius=0.17; visual cylinder length=0 radius=0.17

Commit message: update and try

File: turtlebot_env/resources/obstacle.urdf (robot description, URDF)
Before this commit: robot obstacle, 1 links, 0 joints
Links:
- link base_link: geometry collision cylinder length=0 radius=0; visual cylinder length=0.3 radius=0.17
